Commit message: ouh

File: modelo_robot/urdf/Seguidor_linea_robot.urdf (robot description, URDF)
Before this commit: robot Seguidor_linea_robot, 5 links, 4 joints
Links:
- link Base_castor_link: mass 0.002 -> 0.5
- link Rueda_castor_link: mass 0.00828739992319076 -> 0.0828739992319076
- link Rueda_derecha_link: mass 0.021404 -> 0.1403
- link Rueda_izquierda_link: mass 0.021404 -> 0.1403
- link base_link: mass 0.12859 -> 0.12
Joints:
- joint Base_castor_joint: limit effort=100 velocity=100 -> (none)
- joint Rueda_castor_joint: limit effort=100 velocity=100 -> (none)
- joint Rueda_derecha_joint: limit effort=100 velocity=100 -> (none)
- joint Rueda_izquierda_joint: limit effort=100 velocity=100 -> (none)
